File: hardware/vfd-display/vfd-display.kicad_pcb (KiCad board)
At the start: 2 copper layers, 200 x 65 mm, 48 parts, among them J1 conn_2x3, J2 Conn_01x06_Male, J3 Conn_02x08_Odd_Even, U1 IV-6, U10 IV-6, U11 HV5812, U12 HV5812, U13 IV-6, U14 IV-6, U15 IV-6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

Commit message: tweak placement
Routing:
- net Net-(U4-Pad5): track 0.00 -> 42.9 mm, vias 0 -> 2
- net Net-(U4-Pad6): track 0.00 -> 40.1 mm, vias 0 -> 2
Other:
- net class Default: clearance 0.2 -> 0.127; trace_width 0.25 -> 0.1778; via_dia 0.8 -> 0.889; via_drill 0.4 -> 0.381
- rule trace_clearance: 0.2 -> 0.127
- rule trace_min: 0.2 -> 0.127
- rule via_min_drill: 0.3 -> 0.254
- rule via_min_size: 0.4 -> 0.508

Commit message: Rev 1 design for fab
Parts:
- U16: value LM317 -> LM1084-ADJ
- moved R2 157.5 mm to (245.1, 52.1), turned to 180 degrees
- moved J1 145.6 mm to (221.0, 52.1), turned to 90 degrees
- moved C2 144.3 mm to (54.6, 52.1)
- moved R1 134.8 mm to (245.1, 48.3), turned to 180 degrees
- moved C3 128.7 mm to (54.0, 78.1), turned to 270 degrees
- moved C10 128.0 mm to (104.8, 45.7), turned to 180 degrees
- moved U16 124.8 mm to (104.8, 41.9)
- moved C1 122.8 mm to (93.3, 52.1)
- moved R3 115.9 mm to (196.8, 52.1)
- moved R5 109.9 mm to (210.2, 45.7)
- moved C4 104.1 mm to (112.4, 45.7), turned to 180 degrees
- moved R6 101.5 mm to (182.2, 52.1)
- moved C8 99.6 mm to (238.8, 44.5)
- moved C9 91.6 mm to (183.5, 41.9), turned to 270 degrees
- moved R4 91.2 mm to (140.3, 38.7), turned to 180 degrees
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Connections:
- U16 pad 1: GND -> +1V2
Routing:
- net GND: track 0.00 -> 263.1 mm
- net /GRID: track 0.00 -> 249.6 mm, vias 0 -> 11
- net /STB: track 0.00 -> 207.7 mm, vias 0 -> 5
- net /BL: track 0.00 -> 205.5 mm
- net /CLK: track 0.00 -> 196.0 mm, vias 0 -> 5
- net /DIN: track 0.00 -> 106.6 mm, vias 0 -> 6
- net /D4: track 0.00 -> 104.8 mm, vias 0 -> 6
- net /D1: track 0.00 -> 70.9 mm, vias 0 -> 5
- net +1V2: track 0.00 -> 70.9 mm, vias 0 -> 1
- net /D5: track 0.00 -> 69.4 mm
- net VPP: track 0.00 -> 69.2 mm, vias 0 -> 2
- net /D0: track 0.00 -> 65.2 mm, vias 0 -> 4
- net Net-(J1-Pad5): track 0.00 -> 63.0 mm, vias 0 -> 3
- net /D2: track 0.00 -> 61.5 mm, vias 0 -> 2
- net Net-(U15-Pad10): track 0.00 -> 60.4 mm, vias 0 -> 2
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- added copper zone on B.Cu, net +1V2
- added copper zone on F.Cu, net +5V
- added copper zone on B.Cu, net GND
- added copper zone on F.Cu, net VPP
Other:
- board text added: "12X IV-6 tube mount this side"
- board text added: "2.5V"
- board text added: "2020-07 Rev 1"
- board text added: "25V"
- board text added: "5V"
- board text added: "74LS125"
- board text added: "74LS174"
- board text added: "IV-6 mount on back"
- board text added: "UPCO retro-25 VFD display"
- board text added: "github eshazen/retro-25"
