File: hardware/vfd-display/vfd-display.sch (KiCad schematic (older format))
At the start: 17 parts

Commit message: Preliminary VFD schematic
Parts:
- added C? (x10): C, symbol Device:C
- added C? (x2): 10uF, symbol Device:CP1
- added D? (x2): LED, symbol Device:LED
- added J?: Conn_01x06_Male, symbol Connector:Conn_01x06_Male
- added J?: conn_2x3, symbol Connector_Generic:Conn_02x03_Odd_Even
- added J?: Conn_02x08_Odd_Even, symbol Connector_Generic:Conn_02x08_Odd_Even
- added R? (x2): 470, symbol Device:R_US
- added R?: 100, symbol Device:R_US
- added R?: OMIT, symbol Device:R_US
- added R? (x3): 10k, symbol Device:R_US
- added U?: 74LS125, symbol 74xx:74LS174
- added U? (x5): 74LS125, symbol 74xx:74LS125
- added U?: 74LS125, symbol Regulator_Linear:LM1084-3.3
- U? (x12): value IV-6 -> 74LS125
- U? (x5): value HV5812 -> 74LS125
Connections:
- net labels added: +1V2, +2V5, A0, BL, CLK, D0, D1, D2, D3, D4, D5, D6, D7, F1, F2, GND, GRID, STB, nLED1, nLED2
- wire segments 306 -> 452
Other:
- note added: "5V power for chips, low current"
- note added: "CPU board"
- note added: "Filaments"
- note added: "Jumpers\n"
- note added: "Power"

Commit message: Schematic, footprints, partial placement
Parts:
- C1, C11, C12, C2, C5, C7, C9: renamed from C?; value C -> .01uF; footprint (none) -> Capacitor_THT:C_Disc_D3.8mm_W2.6mm_P2.50mm
- C10: renamed from C?; footprint (none) -> Capacitor_THT:C_Disc_D3.8mm_W2.6mm_P2.50mm; CatNo (none) -> 399-13950-ND
- C3, C6: renamed from C?; value C -> 1uF 50V; footprint (none) -> Capacitor_THT:C_Disc_D3.8mm_W2.6mm_P2.50mm
- C4: renamed from C?; footprint (none) -> Capacitor_THT:C_Disc_D3.8mm_W2.6mm_P2.50mm; CatNo (none) -> 478-7666-ND
- C8: renamed from C?; value C -> 10nF 50V; footprint (none) -> Capacitor_THT:C_Disc_D3.8mm_W2.6mm_P2.50mm
- D1, D2: renamed from D?; footprint (none) -> LED_THT:LED_D3.0mm
- J1: renamed from J?; footprint (none) -> Connector_PinHeader_2.54mm:PinHeader_2x03_P2.54mm_Vertical
- J2: renamed from J?; footprint (none) -> Connector_Molex:Molex_KK-396_A-41791-0006_1x06_P3.96mm_Vertical
- J3: renamed from J?; footprint (none) -> Connector_PinHeader_2.54mm:PinHeader_2x08_P2.54mm_Vertical
- R1, R2, R3, R4, R5, R6, R7: renamed from R?; footprint (none) -> Resistor_THT:R_Axial_DIN0207_L6.3mm_D2.5mm_P10.16mm_Horizontal
- U1, U10, U13, U14, U15, U18, U2, U5, U6, U7, U8, U9: renamed from U?; value 74LS125 -> IV-6; footprint (none) -> iv-6:iv-6v2
- U11, U12, U17, U3, U4: renamed from U?; value 74LS125 -> HV5812; footprint (none) -> Package_DIP:DIP-28_W15.24mm_LongPads
- U16: renamed from U?; value 74LS125 -> LM317; footprint (none) -> Package_TO_SOT_THT:TO-220-3_Vertical
- U19: renamed from U?; footprint (none) -> Package_DIP:DIP-14_W7.62mm_LongPads
- U20: renamed from U?; value 74LS125 -> 74LS174; footprint (none) -> Package_DIP:DIP-16_W7.62mm_LongPads
Other:
- note added: "Retro-25 Calculator"
- note added: "VFD Display Expansion Board"

Commit message: Rev 1 design for fab
Parts:
- removed U16: LM317, Package_TO_SOT_THT:TO-220-3_Vertical, symbol Regulator_Linear:LM1084-3.3
- added U16: LM1084-ADJ, Package_TO_SOT_THT:TO-220-3_Vertical, symbol Regulator_Linear:LM1084-ADJ
Connections:
- wire segments 452 -> 453
Changed lines of the file:
@@
-$EndComp
-$Comp
-L Regulator_Linear:LM1084-3.3 U16
-U 1 1 5F95F319
-P 7700 4250
-F 0 "U16" H 7700 4492 50  0000 C CNN
-F 1 "LM317" H 7700 4401 50  0000 C CNN
-F 2 "Package_TO_SOT_THT:TO-220-3_Vertical" H 7700 4500 50  0001 C CIN
-F 3 "http://www.ti.com/lit/gpn/sn74LS125" H 7700 4250 50  0001 C CNN
-	1    7700 4250
-	1    0    0    -1
 $EndComp
 $Comp
@@
 Wire Wire Line
 	8800 6150 8650 6150
-$Comp
-L power:GND #PWR021
-U 1 1 5FC2D484
-P 7700 4650
-F 0 "#PWR021" H 7700 4400 50  0001 C CNN
-F 1 "GND" H 7705 4477 50  0000 C CNN
-F 2 "" H 7700 4650 50  0001 C CNN
-F 3 "" H 7700 4650 50  0001 C CNN
-	1    7700 4650
-	1    0    0    -1
-$EndComp
-Wire Wire Line
-	7700 4650 7700 4550
 $Comp
 L power:GND #PWR018
@@
 Text Notes 7100 7100 0    100  ~ 0
 VFD Display Expansion Board
+$Comp
+L Regulator_Linear:LM1084-ADJ U16
+U 1 1 5F03E4EB
+P 7700 4250
+F 0 "U16" H 7700 4492 50  0000 C CNN
+F 1 "LM1084-ADJ" H 7700 4401 50  0000 C CNN
+F 2 "Package_TO_SOT_THT:TO-220-3_Vertical" H 7700 4500 50  0001 C CIN
+F 3 "http://www.ti.com/lit/ds/symlink/lm1084.pdf" H 7700 4250 50  0001 C CNN
+	1    7700 4250
+	1    0    0    -1
+$EndComp
+Wire Wire Line
+	8000 4250 8000 4550
+Wire Wire Line
+	8000 4550 7700 4550
+Connection ~ 8000 4250
 $EndSCHEMATC

Commit message: Update schematic PDF
Parts:
- C1, C11, C12, C2, C5, C7, C8, C9: CatNo (none) -> 399-9824-ND
- C3, C6: CatNo (none) -> 399-14394-1-ND
- D1, D2: CatNo (none) -> 1516-1344-ND
- J2: CatNo (none) -> WM4624-ND
- J3: CatNo (none) -> 732-5299-ND
- U11, U12, U17, U3, U4: CatNo (none) -> HV5812P-G-ND
- U16: CatNo (none) -> LM1084IT-ADJ/NOPB-ND
- U19, U20: CatNo (none) -> 296-3664-5-ND
Other:
- note added: "Digit 1"
- note added: "Digit 10"
- note added: "Digit 11"
- note added: "Digit 12"
- note added: "Digit 2"
- note added: "Digit 3"
- note added: "Digit 4"
- note added: "Digit 5"
- note added: "Digit 6"
- note added: "Digit 7"
- note added: "Digit 8"
- note added: "Digit 9"
- note added: "OOPS Adj\nshould be GND"
Changed lines of the file:
@@
 F 2 "Package_DIP:DIP-28_W15.24mm_LongPads" H 2000 850 50  0001 C CNN
 F 3 "http://www.ti.com/lit/gpn/sn74LS125" H 2000 850 50  0001 C CNN
+F 4 "HV5812P-G-ND" V 2350 1000 50  0000 C CNN "CatNo"
 	1    1800 750
 	0    -1   1    0
@@
 F 2 "Package_DIP:DIP-28_W15.24mm_LongPads" H 5050 850 50  0001 C CNN
 F 3 "http://www.ti.com/lit/gpn/sn74LS125" H 5050 850 50  0001 C CNN
+F 4 "HV5812P-G-ND" V 4850 750 50  0001 C CNN "CatNo"
 	1    4850 750
 	0    -1   1    0
@@
 F 2 "Package_DIP:DIP-28_W15.24mm_LongPads" H 2000 4200 50  0001 C CNN
 F 3 "http://www.ti.com/lit/gpn/sn74LS125" H 2000 4200 50  0001 C CNN
+F 4 "HV5812P-G-ND" V 1800 4100 50  0001 C CNN "CatNo"
 	1    1800 4100
 	0    -1   1    0
@@
 F 2 "Package_DIP:DIP-28_W15.24mm_LongPads" H 5050 4200 50  0001 C CNN
 F 3 "http://www.ti.com/lit/gpn/sn74LS125" H 5050 4200 50  0001 C CNN
+F 4 "HV5812P-G-ND" V 4850 4100 50  0001 C CNN "CatNo"
 	1    4850 4100
 	0    -1   1    0
@@
 F 2 "Package_DIP:DIP-28_W15.24mm_LongPads" H 7950 850 50  0001 C CNN
 F 3 "http://www.ti.com/lit/gpn/sn74LS125" H 7950 850 50  0001 C CNN
+F 4 "HV5812P-G-ND" V 7750 750 50  0001 C CNN "CatNo"
 	1    7750 750
 	0    -1   1    0
@@
 F 2 "Capacitor_THT:C_Disc_D3.8mm_W2.6mm_P2.50mm" H 6738 5200 50  0001 C CNN
 F 3 "~" H 6700 5350 50  0001 C CNN
+F 4 "399-9824-ND" V 6550 5550 50  0000 C CNN "CatNo"
 	1    6700 5350
 	1    0    0    -1
@@
 F 2 "Capacitor_THT:C_Disc_D3.8mm_W2.6mm_P2.50mm" H 7088 5200 50  0001 C CNN
 F 3 "~" H 7050 5350 50  0001 C CNN
+F 4 "399-9824-ND" H 7050 5350 50  0001 C CNN "CatNo"
 	1    7050 5350
 	1    0    0    -1
@@
 F 2 "Capacitor_THT:C_Disc_D3.8mm_W2.6mm_P2.50mm" H 7438 5200 50  0001 C CNN
 F 3 "~" H 7400 5350 50  0001 C CNN
+F 4 "399-9824-ND" H 7400 5350 50  0001 C CNN "CatNo"
 	1    7400 5350
 	1    0    0    -1
@@
 F 2 "Capacitor_THT:C_Disc_D3.8mm_W2.6mm_P2.50mm" H 7788 5200 50  0001 C CNN
 F 3 "~" H 7750 5350 50  0001 C CNN
+F 4 "399-9824-ND" H 7750 5350 50  0001 C CNN "CatNo"
 	1    7750 5350
 	1    0    0    -1
@@
 F 2 "Capacitor_THT:C_Disc_D3.8mm_W2.6mm_P2.50mm" H 8138 5200 50  0001 C CNN
 F 3 "~" H 8100 5350 50  0001 C CNN
+F 4 "399-9824-ND" H 8100 5350 50  0001 C CNN "CatNo"
 	1    8100 5350
 	1    0    0    -1
@@
 F 2 "Capacitor_THT:C_Disc_D3.8mm_W2.6mm_P2.50mm" H 7138 5900 50  0001 C CNN
 F 3 "~" H 7100 6050 50  0001 C CNN
+F 4 "399-14394-1-ND" H 7100 5650 50  0000 C CNN "CatNo"
 	1    7100 6050
 	1    0    0    -1
@@
 F 2 "Capacitor_THT:C_Disc_D3.8mm_W2.6mm_P2.50mm" H 7488 5900 50  0001 C CNN
 F 3 "~" H 7450 6050 50  0001 C CNN
+F 4 "399-14394-1-ND" H 7450 6050 50  0001 C CNN "CatNo"
 	1    7450 6050
 	1    0    0    -1
@@
 Wire Wire Line
 	7100 6200 7450 6200
-Text Notes 6900 5100 0    50   ~ 0
+Text Notes 6900 5150 0    50   ~ 0
 5V power for chips, low current
 Text Notes 8450 4300 0    50   ~ 0
@@
 F 2 "Package_DIP:DIP-16_W7.62mm_LongPads" H 10400 1600 50  0001 C CNN
 F 3 "" H 10400 1600 50  0001 C CNN
+F 4 "296-3664-5-ND" H 9950 900 50  0000 C CNN "CatNo"
 	1    10400 1600
 	-1   0    0    -1
@@
 F 2 "Capacitor_THT:C_Disc_D3.8mm_W2.6mm_P2.50mm" H 8488 5200 50  0001 C CNN
 F 3 "~" H 8450 5350 50  0001 C CNN
+F 4 "399-9824-ND" H 8450 5350 50  0001 C CNN "CatNo"
 	1    8450 5350
 	1    0    0    -1
@@
 F 2 "Capacitor_THT:C_Disc_D3.8mm_W2.6mm_P2.50mm" H 8838 5200 50  0001 C CNN
 F 3 "~" H 8800 5350 50  0001 C CNN
+F 4 "399-9824-ND" H 8800 5350 50  0001 C CNN "CatNo"
 	1    8800 5350
 	1    0    0    -1
@@
 F 2 "LED_THT:LED_D3.0mm" H 9350 1200 50  0001 C CNN
 F 3 "~" H 9350 1200 50  0001 C CNN
+F 4 "1516-1344-ND" H 9750 1150 50  0000 C CNN "CatNo"
 	1    9350 1200
 	0    1    1    0
@@
 F 2 "LED_THT:LED_D3.0mm" H 9650 1200 50  0001 C CNN
 F 3 "~" H 9650 1200 50  0001 C CNN
+F 4 "1516-1344-ND" V 9650 1200 50  0001 C CNN "CatNo"
 	1    9650 1200
 	0    1    1    0
@@
 F 2 "Package_DIP:DIP-14_W7.62mm_LongPads" H 10400 3000 50  0001 C CNN
 F 3 "http://www.ti.com/lit/gpn/sn74LS125" H 10400 3000 50  0001 C CNN
+F 4 "296-3664-5-ND" H 10400 3000 50  0001 C CNN "CatNo"
 	1    10400 3000
 	1    0    0    -1
@@
 F 2 "Connector_Molex:Molex_KK-396_A-41791-0006_1x06_P3.96mm_Vertical" H 9850 5850 50  0001 C CNN
 F 3 "~" H 9850 5850 50  0001 C CNN
+F 4 "WM4624-ND" H 9900 5450 50  0000 C CNN "CatNo"
 	1    9850 5850
 	-1   0    0    -1
@@
 F 2 "Package_DIP:DIP-14_W7.62mm_LongPads" H 9450 2450 50  0001 C CNN
 F 3 "http://www.ti.com/lit/gpn/sn74LS125" H 9450 2450 50  0001 C CNN
+F 4 "296-3664-5-ND" V 9700 2450 50  0000 C CNN "CatNo"
 	5    9450 2450
 	1    0    0    -1
@@
 P 9450 1950
 F 0 "#PWR032" H 9450 1800 50  0001 C CNN
-F 1 "+5V" H 9300 2000 50  0000 C CNN
+F 1 "+5V" H 9550 1950 50  0000 C CNN
 F 2 "" H 9450 1950 50  0001 C CNN
 F 3 "" H 9450 1950 50  0001 C CNN
@@
 F 2 "Capacitor_THT:C_Disc_D3.8mm_W2.6mm_P2.50mm" H 7988 6000 50  0001 C CNN
 F 3 "~" H 7950 6150 50  0001 C CNN
+F 4 "399-9824-ND" H 7950 6150 50  0001 C CNN "CatNo"
 	1    7950 6150
 	1    0    0    -1
@@
 F 2 "Package_DIP:DIP-14_W7.62mm_LongPads" H 10400 3550 50  0001 C CNN
 F 3 "http://www.ti.com/lit/gpn/sn74LS125" H 10400 3550 50  0001 C CNN
+F 4 "296-3664-5-ND" H 10400 3550 50  0001 C CNN "CatNo"
 	2    10400 3550
 	1    0    0    -1
@@
 F 2 "Package_DIP:DIP-14_W7.62mm_LongPads" H 10400 4100 50  0001 C CNN
 F 3 "http://www.ti.com/lit/gpn/sn74LS125" H 10400 4100 50  0001 C CNN
+F 4 "296-3664-5-ND" H 10400 4100 50  0001 C CNN "CatNo"
 	3    10400 4100
 	1    0    0    -1
@@
 F 2 "Package_DIP:DIP-14_W7.62mm_LongPads" H 10400 4650 50  0001 C CNN
 F 3 "http://www.ti.com/lit/gpn/sn74LS125" H 10400 4650 50  0001 C CNN
+F 4 "296-3664-5-ND" H 10400 4650 50  0001 C CNN "CatNo"
 	4    10400 4650
 	1    0    0    -1
@@
 F 2 "Connector_PinHeader_2.54mm:PinHeader_2x08_P2.54mm_Vertical" H 10500 5850 50  0001 C CNN
 F 3 "~" H 10500 5850 50  0001 C CNN
+F 4 "732-5299-ND" H 10550 5350 50  0000 C CNN "CatNo"
 	1    10500 5850
 	1    0    0    -1
@@
 F 2 "Package_TO_SOT_THT:TO-220-3_Vertical" H 7700 4500 50  0001 C CIN
 F 3 "http://www.ti.com/lit/ds/symlink/lm1084.pdf" H 7700 4250 50  0001 C CNN
+F 4 "LM1084IT-ADJ/NOPB-ND" H 7700 4650 50  0000 C CNN "CatNo"
 	1    7700 4250
 	1    0    0    -1
@@
 	8000 4550 7700 4550
 Connection ~ 8000 4250
+Text Notes 8700 3500 0    50   ~ 0
+Digit 1
+Text Notes 7500 3500 0    50   ~ 0
+Digit 2
+Text Notes 6200 3500 0    50   ~ 0
+Digit 3
+Text Notes 4950 3500 0    50   ~ 0
+Digit 4
+Text Notes 3800 3500 0    50   ~ 0
+Digit 5
+Text Notes 2650 3500 0    50   ~ 0
+Digit 6
+Text Notes 1500 3500 0    50   ~ 0
+Digit 7
+Text Notes 6200 6850 0    50   ~ 0
+Digit 8
+Text Notes 4950 6850 0    50   ~ 0
+Digit 9
+Text Notes 3800 6850 0    50   ~ 0
+Digit 10
+Text Notes 2650 6850 0    50   ~ 0
+Digit 11
+Text Notes 1500 6850 0    50   ~ 0
+Digit 12
+Text Notes 7350 4800 0    50   ~ 0
+OOPS Adj\nshould be GND
 $EndSCHEMATC
