File: hardware/psu/trunk/psu.kicad_pcb (KiCad board)
At the start: 2 copper layers, 127 x 50.8 mm, 29 parts, among them J1 Conn_01x02_Male, J2 Conn_01x04_Male, J3 Conn_01x06_Male, J4 Conn_01x02_Male, Q1 2N3904, Q2 2N3904, Q3 2N3906, Q4 2N3906, Q5 IRF540N, Q6 IRF540N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

Commit message: ordered PCBs
Other:
- board text added: "+ - 9V in"
- board text added: "+18V"
- board text added: "+2.5V"
- board text added: "- +"
- board text added: "9V to CPU"
- board text added: "CTRL in"
- board text added: "Fil"
- board text added: "GND"
- board text added: "NC"
- board text added: "UPCO Retro-25 Power Supply"
- board text added: "Vpp"
- board text added: "en18"
- board text added: "en2.5"
- board text added: "to VFD"
