File: hardware/cpu/RevA/cpu.sch (KiCad schematic (older format))
At the start: 49 parts, among them J1 hdr_2x8, J2 Conn_01x06, J3 hdr_2x8, J5 Conn_01x02, SW1 SW_Push, U1 74AS74, U13 74LS32, U16 uA7805, U17 74AS74, U2 74LS374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

Commit message: fix bugs in bootloader, make umon base control by makefile
Parts:
- RN1: CatNo (none) -> 4609X-AP1-103LFCT-ND
Changed lines of the file:
@@
 EESchema Schematic File Version 4
-LIBS:cpu-cache
-EELAYER 26 0
+EELAYER 30 0
 EELAYER END
 $Descr A 11000 8500
@@
 F 2 "Resistor_THT:R_Array_SIP9" V 4150 4300 50  0001 C CNN
 F 3 "" H 3675 4300 50  0001 C CNN
+F 4 "4609X-AP1-103LFCT-ND" H 3725 4625 50  0000 C CNN "CatNo"
 	1    3675 4300
 	0    1    1    0
